File: board/USBPD.kicad_pcb (KiCad board)
At the start: 2 copper layers, 21.5 x 19 mm, 22 parts, among them J1 USB_C_Receptacle, J2 POWER, J3 UDPI, J4 UART, Q1 PMOS, Q2 PMOS, Q3 PMOS, U1 AP7384, U2 FUSB302, U3 ATtiny1626-M

Commit message: update pcb
Connections:
- D1 pad 1: GND -> Net-(D1-Pad1)
- D1 pad 3: Net-(D1-Pad3) -> GND
- R1 pad 2: Net-(D1-Pad3) -> Net-(D1-Pad1)
- U2 pad 10: Net-(D1-Pad3) -> Net-(D1-Pad1)
- U2 pad 11: Net-(D1-Pad3) -> Net-(D1-Pad1)
Routing:
- net Net-(D1-Pad1): track 0.00 -> 8.02 mm
- net Net-(D1-Pad3): track 6.85 -> 0.00 mm
Changed lines of the file:
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@@
   (net 31 "unconnected-(U3-Pad8)")
   (net 32 "unconnected-(U3-Pad9)")
-  (net 33 "Net-(D1-Pad3)")
+  (net 33 "Net-(D1-Pad1)")
   (net 34 "Net-(D1-Pad2)")
   (net 35 "Net-(Q2-Pad4)")
@@
       (net 8 "Net-(J1-PadA5)") (pintype "passive"))
     (pad "2" smd roundrect (at 0.825 0) (size 0.8 0.95) (layers "F.Cu" "F.Paste" "F.Mask") (roundrect_rratio 0.25)
-      (net 33 "Net-(D1-Pad3)") (pintype "passive"))
+      (net 33 "Net-(D1-Pad1)") (pintype "passive"))
     (model "${KICAD6_3DMODEL_DIR}/Resistor_SMD.3dshapes/R_0603_1608Metric.wrl"
       (offset (xyz 0 0 0))
@@
     (fp_line (start -0.65 1.45) (end -0.65 -1.125) (layer "F.Fab") (width 0.1))
     (pad "1" smd roundrect (at -0.9375 -0.95) (size 1.475 0.6) (layers "F.Cu" "F.Paste" "F.Mask") (roundrect_rratio 0.25)
-      (net 2 "GND") (pinfunction "A") (pintype "passive"))
+      (net 33 "Net-(D1-Pad1)") (pinfunction "K") (pintype "passive"))
     (pad "2" smd roundrect (at -0.9375 0.95) (size 1.475 0.6) (layers "F.Cu" "F.Paste" "F.Mask") (roundrect_rratio 0.25)
       (net 34 "Net-(D1-Pad2)") (pinfunction "K") (pintype "passive"))
     (pad "3" smd roundrect (at 0.9375 0) (size 1.475 0.6) (layers "F.Cu" "F.Paste" "F.Mask") (roundrect_rratio 0.25)
-      (net 33 "Net-(D1-Pad3)") (pinfunction "K") (pintype "passive"))
+      (net 2 "GND") (pinfunction "A") (pintype "passive"))
     (model "${KICAD6_3DMODEL_DIR}/Package_TO_SOT_SMD.3dshapes/SOT-23.wrl"
       (offset (xyz 0 0 0))
@@
       (net 2 "GND") (pinfunction "GND") (pintype "passive"))
     (pad "10" smd roundrect (at 1.2625 -0.5 90) (size 0.675 0.25) (layers "F.Cu" "F.Paste" "F.Mask") (roundrect_rratio 0.25)
-      (net 33 "Net-(D1-Pad3)") (pinfunction "CC1") (pintype "bidirectional"))
+      (net 33 "Net-(D1-Pad1)") (pinfunction "CC1") (pintype "bidirectional"))
     (pad "11" smd roundrect (at 0.75 -1.2625 90) (size 0.25 0.675) (layers "F.Cu" "F.Paste" "F.Mask") (roundrect_rratio 0.25)
-      (net 33 "Net-(D1-Pad3)") (pinfunction "CC1") (pintype "bidirectional"))
+      (net 33 "Net-(D1-Pad1)") (pinfunction "CC1") (pintype "bidirectional"))
     (pad "12" smd roundrect (at 0.25 -1.2625 90) (size 0.25 0.675) (layers "F.Cu" "F.Paste" "F.Mask") (roundrect_rratio 0.25)
       (net 6 "+5V") (pinfunction "VCONN") (pintype "power_in"))
@@
   (segment (start 61.3 110.9) (end 62.3 109.9) (width 0.15) (layer "B.Cu") (net 27))
   (segment (start 64.4 109.9) (end 64.9 110.4) (width 0.15) (layer "B.Cu") (net 27))
+  (segment (start 69.01 110.23) (end 67.8125 109.0325) (width 0.15) (layer "F.Cu") (net 33))
+  (segment (start 68.575 112.5) (end 69.01 112.065) (width 0.15) (layer "F.Cu") (net 33))
   (segment (start 69.0625 112.9875) (end 68.575 112.5) (width 0.2) (layer "F.Cu") (net 33))
+  (segment (start 67.8125 109.0325) (end 67.8125 108.55) (width 0.15) (layer "F.Cu") (net 33))
   (segment (start 70.4875 112.9875) (end 69.0625 112.9875) (width 0.2) (layer "F.Cu") (net 33))
-  (segment (start 68.575 112.5) (end 69.6875 111.3875) (width 0.2) (layer "F.Cu") (net 33))
+  (segment (start 69.01 112.065) (end 69.01 110.23) (width 0.15) (layer "F.Cu") (net 33))
   (segment (start 71.25 112.9875) (end 70.4875 112.9875) (width 0.2) (layer "F.Cu") (net 33))
   (segment (start 70.4875 113.5) (end 70.4875 112.9875) (width 0.2) (layer "F.Cu") (net 33))
-  (segment (start 69.6875 111.3875) (end 69.6875 109.5) (width 0.2) (layer "F.Cu") (net 33))
   (segment (start 70.4875 115.5125) (end 68.7375 115.5125) (width 0.2) (layer "F.Cu") (net 34))
   (segment (start 70.4875 115) (end 70.4875 115.5125) (width 0.2) (layer "F.Cu") (net 34))

Commit message: use LVL translator for switch
Parts:
- added Q4: NMOS, Package_TO_SOT_SMD:SOT-23, B.Cu at (73.6, 119.5)
Connections:
- Q2 pad 3: /SRC -> Net-(Q2-Pad3)
- Q3 pad 3: /SRC -> Net-(Q2-Pad3)
- R3 pad 2: /SRC -> Net-(Q2-Pad3)
Routing:
- net Net-(Q2-Pad3): track 0.00 -> 7.20 mm, vias 0 -> 2
- net +3.3V: track 32.3 -> 34.5 mm
- net +5V: track 28.5 -> 29.1 mm
- net /SRC: track 36.2 -> 35.7 mm, vias 4 -> 2
